File: schematic/rover/power_supply.kicad_sch (KiCad schematic)
At the start: 0 parts

Commit message: Complete power board and motor wiring
Parts:
- added C3, C4: 10uF, symbol Device:C
- added D1, D3: 1N4733A, Diode_THT:D_DO-41_SOD81_P10.16mm_Horizontal, symbol Diode:1N47xxA
- added D2, D4: 1N5820, Diode_THT:D_DO-201AD_P15.24mm_Horizontal, symbol Diode:1N5820
- added F1: 500mA, symbol Device:Fuse
- added F2: 5A, symbol Device:Fuse
Connections:
- new net: C3.1, D1.1 (K), D2.2 (A), F1.1
- new net 5V_FlightController: F2.2
- new net 5V_HighPowerOutput: D4.1 (K)
- new net 5V_LowPowerOutput: D2.1 (K)
- new net 5V_MotorController: F1.2
- new net 5V_RaspberryPi: C4.1, D3.1 (K), D4.2 (A), F2.1
- new net GND: C3.2, C4.2, D1.2 (A), D3.2 (A)
