File: schematic/rover/rover.kicad_pcb (KiCad board)
At the start: 2 copper layers, 20 parts, among them J1 Conn_02x05_Odd_Even, J10 Conn_01x05_Pin, J11 Conn_01x05_Pin, J12 Conn_01x04_Pin, J13 Conn_02x05_Odd_Even, J14 Conn_01x04_Pin, J15 Conn_01x03_Socket, J16 Conn_01x05_Pin, J17 Conn_01x05_Pin, J2 Conn_02x05_Odd_Even, J3 Conn_02x05_Odd_Even, J4 Conn_01x03_Socket, J5 Conn_02x05_Odd_Even, J6 Conn_01x04_Pin, J7 Conn_02x05_Odd_Even, J8 Conn_01x04_Pin, J9 Conn_01x03_Socket, U1 Pico

Commit message: Complete motor controller schematic
Parts:
- added U2: Pico, MCU_RaspberryPi_and_Boards:RPi_Pico_SMD_TH, F.Cu at (71.1, 63.5)
- added U3: Pico, MCU_RaspberryPi_and_Boards:RPi_Pico_SMD_TH, F.Cu at (315.0, 71.1)
- added U4: ACS711xEXLT-31AB, Sensor_Current:Allegro_QFN-12-10-1EP_3x3mm_P0.5mm, F.Cu at (109.4, 48.3)
- added U5: ACS711xEXLT-31AB, Sensor_Current:Allegro_QFN-12-10-1EP_3x3mm_P0.5mm, F.Cu at (346.6, 79.0)
- added U6: ACS711xEXLT-31AB, Sensor_Current:Allegro_QFN-12-10-1EP_3x3mm_P0.5mm, F.Cu at (110.5, 78.2)
- added U7: ACS711xEXLT-31AB, Sensor_Current:Allegro_QFN-12-10-1EP_3x3mm_P0.5mm, F.Cu at (351.6, 50.0)
- J10, J16: value Conn_01x05_Pin -> Right_Current_Sense
- J11, J17: value Conn_01x05_Pin -> Left_Current_Sense
- J12, J6: value Conn_01x04_Pin -> Left_Encoder
- J14, J8: value Conn_01x04_Pin -> Right_Encoder
- moved J16 350.9 mm to (347.8, 60.7), turned to 90 degrees
- moved J17 348.5 mm to (342.7, 93.7), turned to 90 degrees
- moved J13 275.9 mm to (279.4, 66.0)
- moved J12 273.2 mm to (277.3, 88.9)
- moved J14 273.2 mm to (281.9, 88.9)
- moved J1 266.0 mm to (113.0, 212.1)
- moved J3 266.0 mm to (97.8, 245.1)
- moved J15 265.8 mm to (281.9, 48.3)
- moved C2 263.9 mm to (132.1, 265.4)
- moved C1 260.4 mm to (142.3, 250.2)
- moved J4 218.4 mm to (133.3, 224.8)
- moved U1 210.2 mm to (177.8, 243.8)
- moved J2 152.6 mm to (144.8, 198.1)
- moved J10 146.9 mm to (104.1, 57.2), turned to 90 degrees
- moved J11 145.1 mm to (104.5, 87.3), turned to 90 degrees
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Connections:
- J10 pad 1: unconnected-(J10-Pin_1-Pad1) -> GND
- J10 pad 2: unconnected-(J10-Pin_2-Pad2) -> GND
- J10 pad 3: unconnected-(J10-Pin_3-Pad3) -> +3.3V
- J10 pad 4: unconnected-(J10-Pin_4-Pad4) -> Net-(J10-Pin_4)
- J11 pad 1: unconnected-(J11-Pin_1-Pad1) -> GND
- J11 pad 2: unconnected-(J11-Pin_2-Pad2) -> GND
- J11 pad 3: unconnected-(J11-Pin_3-Pad3) -> +3.3V
- J11 pad 4: unconnected-(J11-Pin_4-Pad4) -> Net-(J11-Pin_4)
- J12 pad 1: unconnected-(J12-Pin_1-Pad1) -> /low level control/motor_controller_rear/OUTB_L__Green
- J12 pad 2: unconnected-(J12-Pin_2-Pad2) -> GND
- J12 pad 3: unconnected-(J12-Pin_3-Pad3) -> +3.3V
- J12 pad 4: unconnected-(J12-Pin_4-Pad4) -> /low level control/motor_controller_rear/OUTA_L__Blue
- J13 pad 10: unconnected-(J13-Pin_10-Pad10) -> /low level control/motor_controller_rear/Central_Hub__RX
- J13 pad 2: unconnected-(J13-Pin_2-Pad2) -> GND
- J13 pad 4: unconnected-(J13-Pin_4-Pad4) -> /low level control/motor_controller_rear/OUTB_L__Green
- J13 pad 6: unconnected-(J13-Pin_6-Pad6) -> /low level control/motor_controller_rear/OUTA_L__Blue
- J13 pad 7: unconnected-(J13-Pin_7-Pad7) -> /low level control/motor_controller_rear/OUTA_R__Blue
- J13 pad 8: unconnected-(J13-Pin_8-Pad8) -> /low level control/motor_controller_rear/Central_Hub__TX
- J13 pad 9: unconnected-(J13-Pin_9-Pad9) -> /low level control/motor_controller_rear/OUTB_R__Green
- J14 pad 1: unconnected-(J14-Pin_1-Pad1) -> /low level control/motor_controller_rear/OUTB_R__Green
- J14 pad 2: unconnected-(J14-Pin_2-Pad2) -> GND
- J14 pad 3: unconnected-(J14-Pin_3-Pad3) -> +3.3V
- J14 pad 4: unconnected-(J14-Pin_4-Pad4) -> /low level control/motor_controller_rear/OUTA_R__Blue
- J15 pad 2: unconnected-(J15-Pin_2-Pad2) -> /low level control/motor_controller_rear/Sabertooth__TX
- J16 pad 1: unconnected-(J16-Pin_1-Pad1) -> GND
- J16 pad 2: unconnected-(J16-Pin_2-Pad2) -> GND
- J16 pad 3: unconnected-(J16-Pin_3-Pad3) -> +3.3V
- J16 pad 4: unconnected-(J16-Pin_4-Pad4) -> Net-(J16-Pin_4)
- J17 pad 1: unconnected-(J17-Pin_1-Pad1) -> GND
- J17 pad 2: unconnected-(J17-Pin_2-Pad2) -> GND
- J17 pad 3: unconnected-(J17-Pin_3-Pad3) -> +3.3V
- J17 pad 4: unconnected-(J17-Pin_4-Pad4) -> Net-(J17-Pin_4)
- J6 pad 1: unconnected-(J6-Pin_1-Pad1) -> /low level control/motor_controller_front/OUTB_L__Green
- J6 pad 2: unconnected-(J6-Pin_2-Pad2) -> GND
- J6 pad 3: unconnected-(J6-Pin_3-Pad3) -> +3.3V
- J6 pad 4: unconnected-(J6-Pin_4-Pad4) -> /low level control/motor_controller_front/OUTA_L__Blue
- J7 pad 10: unconnected-(J7-Pin_10-Pad10) -> /low level control/motor_controller_front/Central_Hub__RX
- J7 pad 2: unconnected-(J7-Pin_2-Pad2) -> GND
- J7 pad 4: unconnected-(J7-Pin_4-Pad4) -> /low level control/motor_controller_front/OUTB_L__Green
- J7 pad 6: unconnected-(J7-Pin_6-Pad6) -> /low level control/motor_controller_front/OUTA_L__Blue
- J7 pad 7: unconnected-(J7-Pin_7-Pad7) -> /low level control/motor_controller_front/OUTA_R__Blue
- J7 pad 8: unconnected-(J7-Pin_8-Pad8) -> /low level control/motor_controller_front/Central_Hub__TX
- J7 pad 9: unconnected-(J7-Pin_9-Pad9) -> /low level control/motor_controller_front/OUTB_R__Green
- J8 pad 1: unconnected-(J8-Pin_1-Pad1) -> /low level control/motor_controller_front/OUTB_R__Green
- J8 pad 2: unconnected-(J8-Pin_2-Pad2) -> GND
- J8 pad 3: unconnected-(J8-Pin_3-Pad3) -> +3.3V
- J8 pad 4: unconnected-(J8-Pin_4-Pad4) -> /low level control/motor_controller_front/OUTA_R__Blue
- J9 pad 2: unconnected-(J9-Pin_2-Pad2) -> /low level control/motor_controller_front/Sabertooth__TX

Commit message: Arrange components following the stripboard layout
Parts:
- removed J4: Conn_01x03_Socket, Connector_PinHeader_2.54mm:PinHeader_1x03_P2.54mm_Vertical
- added D1: 1N4733A, Diode_THT:D_DO-41_SOD81_P10.16mm_Horizontal, F.Cu at (-63.5, 112.6)
- added D2: 1N5820, Diode_THT:D_DO-201AD_P15.24mm_Horizontal, F.Cu at (-63.0, 100.3)
- added D3: 1N4733A, Diode_THT:D_DO-41_SOD81_P10.16mm_Horizontal, F.Cu at (-63.5, 116.8)
- added D4: 1N5820, Diode_THT:D_DO-201AD_P15.24mm_Horizontal, F.Cu at (-63.0, 107.1)
- added J18: Conn_01x04_Socket, Connector_PinHeader_2.54mm:PinHeader_1x04_P2.54mm_Vertical, F.Cu at (198.1, 218.4)
- added Q1: BC547, Package_TO_SOT_THT:TO-92_Inline, F.Cu at (203.0, 245.3)
- added R1: 100k, Resistor_THT:R_Axial_DIN0207_L6.3mm_D2.5mm_P5.08mm_Vertical, F.Cu at (193.0, 246.4)
- C1, C2: value C -> 3.3n; footprint Capacitor_THT:C_Disc_D7.5mm_W5.0mm_P7.50mm -> Capacitor_THT:C_Disc_D5.0mm_W2.5mm_P5.00mm
- J1: value Conn_02x05_Odd_Even -> Front_Wheel_Conn
- J2: value Conn_02x05_Odd_Even -> Rear_Wheel_Conn
- J3: value Conn_02x05_Odd_Even -> Flight_Controller_Conn
- J5: value Conn_02x05_Odd_Even -> Receiver_Conn
- moved J5 119.3 mm to (203.2, 256.5)
- moved J3 63.3 mm to (160.0, 256.5)
- moved J1 52.8 mm to (160.0, 236.2)
- moved C2 33.0 mm to (165.1, 266.6), turned to 90 degrees
- moved C1 30.2 mm to (167.6, 266.6), turned to 90 degrees
- moved J2 25.4 mm to (160.0, 218.4)
- moved U6 19.7 mm to (91.0, 81.0), turned to -90 degrees
- moved J11 18.2 mm to (86.4, 88.9)
- moved J14 18.0 mm to (299.7, 86.4)
- moved J10 17.8 mm to (86.4, 58.4)
- moved J6 17.8 mm to (48.3, 81.3)
- moved U4 17.7 mm to (91.9, 50.7)
- moved J13 15.5 mm to (294.6, 63.5)
- moved U7 15.3 mm to (337.6, 56.2), turned to -90 degrees
- moved J16 15.3 mm to (332.7, 63.5)
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Connections:
- net /low level control/motor_controller_front/Left_Motor_Driver_Output renamed /low level control/Sabertooth_front/M1A
- net /low level control/motor_controller_front/Left_Motor_Terminal renamed /low level control/Sabertooth_front/M1B
- net /low level control/motor_controller_front/Right_Motor_Driver_Output renamed /low level control/Sabertooth_front/M2B
- net /low level control/motor_controller_front/Right_Motor_Terminal renamed /low level control/Sabertooth_front/M2A
- net /low level control/motor_controller_front/Sabertooth__TX renamed /low level control/Sabertooth_front/S1
- net /low level control/motor_controller_rear/Left_Motor_Driver_Output renamed /low level control/Sabertooth_rear/M1A
- net /low level control/motor_controller_rear/Left_Motor_Terminal renamed /low level control/Sabertooth_rear/M1B
- net /low level control/motor_controller_rear/Right_Motor_Driver_Output renamed /low level control/Sabertooth_rear/M2B
- net /low level control/motor_controller_rear/Right_Motor_Terminal renamed /low level control/Sabertooth_rear/M2A
- net /low level control/motor_controller_rear/Sabertooth__TX renamed /low level control/Sabertooth_rear/S1
- C1 pad 1: unconnected-(C1-Pad1) -> /low level control/central_hub/FC__Throttle_Left
- C2 pad 1: unconnected-(C2-Pad1) -> /low level control/central_hub/FC__Throttle_Right
- J1 pad 10: unconnected-(J1-Pin_10-Pad10) -> /low level control/central_hub/Front_Controller__TX
- J1 pad 2: unconnected-(J1-Pin_2-Pad2) -> GND
- J1 pad 4: unconnected-(J1-Pin_4-Pad4) -> /low level control/central_hub/OUTB_Right__Front
- J1 pad 6: unconnected-(J1-Pin_6-Pad6) -> /low level control/central_hub/OUTA_Right__Front
- J1 pad 7: unconnected-(J1-Pin_7-Pad7) -> /low level control/central_hub/OUTA_Left__Front
- J1 pad 8: unconnected-(J1-Pin_8-Pad8) -> /low level control/central_hub/Front_Controller__RX
- J1 pad 9: unconnected-(J1-Pin_9-Pad9) -> /low level control/central_hub/OUTB_Left__Front
- J12 pad 1: /low level control/motor_controller_rear/OUTB_L__Green -> /low level control/central_hub/OUTB_Left__Rear
- J12 pad 4: /low level control/motor_controller_rear/OUTA_L__Blue -> /low level control/central_hub/OUTA_Left__Rear
- J13 pad 10: /low level control/motor_controller_rear/Central_Hub__RX -> /low level control/central_hub/Rear_Controller__TX
- J13 pad 4: /low level control/motor_controller_rear/OUTB_L__Green -> /low level control/central_hub/OUTB_Right__Rear
- J13 pad 6: /low level control/motor_controller_rear/OUTA_L__Blue -> /low level control/central_hub/OUTA_Right__Rear
- J13 pad 7: /low level control/motor_controller_rear/OUTA_R__Blue -> /low level control/central_hub/OUTA_Left__Rear
- J13 pad 8: /low level control/motor_controller_rear/Central_Hub__TX -> /low level control/central_hub/Rear_Controller__RX
- J13 pad 9: /low level control/motor_controller_rear/OUTB_R__Green -> /low level control/central_hub/OUTB_Left__Rear
- J14 pad 1: /low level control/motor_controller_rear/OUTB_R__Green -> /low level control/central_hub/OUTB_Right__Rear
- J14 pad 4: /low level control/motor_controller_rear/OUTA_R__Blue -> /low level control/central_hub/OUTA_Right__Rear
- J2 pad 10: unconnected-(J2-Pin_10-Pad10) -> /low level control/central_hub/Rear_Controller__TX
- J2 pad 2: unconnected-(J2-Pin_2-Pad2) -> GND
- J2 pad 4: unconnected-(J2-Pin_4-Pad4) -> /low level control/central_hub/OUTB_Right__Rear
- J2 pad 6: unconnected-(J2-Pin_6-Pad6) -> /low level control/central_hub/OUTA_Right__Rear
- J2 pad 7: unconnected-(J2-Pin_7-Pad7) -> /low level control/central_hub/OUTA_Left__Rear
- J2 pad 8: unconnected-(J2-Pin_8-Pad8) -> /low level control/central_hub/Rear_Controller__RX
- J2 pad 9: unconnected-(J2-Pin_9-Pad9) -> /low level control/central_hub/OUTB_Left__Rear
- J3 pad 1: unconnected-(J3-Pin_1-Pad1) -> /low level control/central_hub/FC__SBUS
- J3 pad 10: unconnected-(J3-Pin_10-Pad10) -> /low level control/central_hub/FC__Throttle_Right
- J3 pad 2: unconnected-(J3-Pin_2-Pad2) -> /low level control/central_hub/OUTB_Right__Rear
- J3 pad 3: unconnected-(J3-Pin_3-Pad3) -> /low level control/central_hub/OUTA_Left__Rear
- J3 pad 4: unconnected-(J3-Pin_4-Pad4) -> /low level control/central_hub/OUTA_Right__Rear
- J3 pad 5: unconnected-(J3-Pin_5-Pad5) -> /low level control/central_hub/OUTB_Left__Rear
- J3 pad 6: unconnected-(J3-Pin_6-Pad6) -> GND
- J3 pad 7: unconnected-(J3-Pin_7-Pad7) -> /low level control/central_hub/Flight_Controller__RX
- J3 pad 8: unconnected-(J3-Pin_8-Pad8) -> /low level control/central_hub/FC__Throttle_Left
- J3 pad 9: unconnected-(J3-Pin_9-Pad9) -> /low level control/central_hub/Flight_Controller__TX
- J5 pad 1: unconnected-(J5-Pin_1-Pad1) -> /low level control/central_hub/FC__SBUS
- J5 pad 2: unconnected-(J5-Pin_2-Pad2) -> /low level control/central_hub/Receiver__PPM
- J5 pad 3: unconnected-(J5-Pin_3-Pad3) -> +3.3V
- J5 pad 5: unconnected-(J5-Pin_5-Pad5) -> GND
- J6 pad 1: /low level control/motor_controller_front/OUTB_L__Green -> /low level control/central_hub/OUTB_Left__Front
- J6 pad 4: /low level control/motor_controller_front/OUTA_L__Blue -> /low level control/central_hub/OUTA_Left__Front
- J7 pad 10: /low level control/motor_controller_front/Central_Hub__RX -> /low level control/central_hub/Front_Controller__TX
- J7 pad 4: /low level control/motor_controller_front/OUTB_L__Green -> /low level control/central_hub/OUTB_Right__Front
- J7 pad 6: /low level control/motor_controller_front/OUTA_L__Blue -> /low level control/central_hub/OUTA_Right__Front
- J7 pad 7: /low level control/motor_controller_front/OUTA_R__Blue -> /low level control/central_hub/OUTA_Left__Front
- J7 pad 8: /low level control/motor_controller_front/Central_Hub__TX -> /low level control/central_hub/Front_Controller__RX
- J7 pad 9: /low level control/motor_controller_front/OUTB_R__Green -> /low level control/central_hub/OUTB_Left__Front
- J8 pad 1: /low level control/motor_controller_front/OUTB_R__Green -> /low level control/central_hub/OUTB_Right__Front
- J8 pad 4: /low level control/motor_controller_front/OUTA_R__Blue -> /low level control/central_hub/OUTA_Right__Front
- U1 pad 1: unconnected-(U1-GPIO0-Pad1) -> /low level control/central_hub/Front_Controller__TX
- U1 pad 11: unconnected-(U1-GPIO8-Pad11) -> /low level control/central_hub/Rear_Controller__TX
- U1 pad 12: unconnected-(U1-GPIO9-Pad12) -> /low level control/central_hub/Rear_Controller__RX
- U1 pad 13: unconnected-(U1-GND-Pad13) -> GND
- U1 pad 14: unconnected-(U1-GPIO10-Pad14) -> /low level control/central_hub/OUTA_Left__Rear
- U1 pad 15: unconnected-(U1-GPIO11-Pad15) -> /low level control/central_hub/OUTB_Left__Rear
- U1 pad 16: unconnected-(U1-GPIO12-Pad16) -> /low level control/central_hub/OUTB_Right__Rear
- U1 pad 17: unconnected-(U1-GPIO13-Pad17) -> /low level control/central_hub/OUTA_Right__Rear
- U1 pad 18: unconnected-(U1-GND-Pad18) -> GND
- U1 pad 19: unconnected-(U1-GPIO14-Pad19) -> /low level control/central_hub/FC__Throttle_Left
- U1 pad 2: unconnected-(U1-GPIO1-Pad2) -> /low level control/central_hub/Front_Controller__RX
- U1 pad 20: unconnected-(U1-GPIO15-Pad20) -> /low level control/central_hub/FC__Throttle_Right
- U1 pad 21: unconnected-(U1-GPIO16-Pad21) -> /low level control/central_hub/Flight_Controller__TX
- U1 pad 22: unconnected-(U1-GPIO17-Pad22) -> /low level control/central_hub/Flight_Controller__RX
- U1 pad 27: unconnected-(U1-GPIO21-Pad27) -> /low level control/central_hub/Receiver__PPM
- U1 pad 29: unconnected-(U1-GPIO22-Pad29) -> Net-(U1-GPIO22)
- U1 pad 3: unconnected-(U1-GND-Pad3) -> GND
- U1 pad 32: unconnected-(U1-GPIO27_ADC1-Pad32) -> /low level control/central_hub/NeoPixelRGB
- U1 pad 4: unconnected-(U1-GPIO2-Pad4) -> /low level control/central_hub/OUTB_Right__Front
- U1 pad 5: unconnected-(U1-GPIO3-Pad5) -> /low level control/central_hub/OUTA_Right__Front
- U1 pad 6: unconnected-(U1-GPIO4-Pad6) -> /low level control/central_hub/OUTB_Left__Front
- U1 pad 7: unconnected-(U1-GPIO5-Pad7) -> /low level control/central_hub/OUTA_Left__Front
- U1 pad 8: unconnected-(U1-GND-Pad8) -> GND
- U2 pad 16: /low level control/motor_controller_front/OUTA_L__Blue -> /low level control/central_hub/OUTA_Left__Front
- U2 pad 17: /low level control/motor_controller_front/OUTB_L__Green -> /low level control/central_hub/OUTB_Left__Front
- U2 pad 19: /low level control/motor_controller_front/OUTB_R__Green -> /low level control/central_hub/OUTB_Right__Front
- U2 pad 20: /low level control/motor_controller_front/OUTA_R__Blue -> /low level control/central_hub/OUTA_Right__Front
- U2 pad 39: +5V -> /low level control/+5V_in
- U2 pad 6: /low level control/motor_controller_front/Central_Hub__TX -> /low level control/central_hub/Front_Controller__RX
- U2 pad 7: /low level control/motor_controller_front/Central_Hub__RX -> /low level control/central_hub/Front_Controller__TX
- U3 pad 16: /low level control/motor_controller_rear/OUTA_L__Blue -> /low level control/central_hub/OUTA_Left__Rear
- U3 pad 17: /low level control/motor_controller_rear/OUTB_L__Green -> /low level control/central_hub/OUTB_Left__Rear
- U3 pad 19: /low level control/motor_controller_rear/OUTB_R__Green -> /low level control/central_hub/OUTB_Right__Rear
- U3 pad 20: /low level control/motor_controller_rear/OUTA_R__Blue -> /low level control/central_hub/OUTA_Right__Rear
- U3 pad 39: +5V -> /low level control/+5V_in
- U3 pad 6: /low level control/motor_controller_rear/Central_Hub__TX -> /low level control/central_hub/Rear_Controller__RX
- U3 pad 7: /low level control/motor_controller_rear/Central_Hub__RX -> /low level control/central_hub/Rear_Controller__TX
